Commit message: included three Hokuyo and one Velodyne LIDAR

File: urdf/robot.urdf (robot description, URDF)
Before this commit: robot insert_robot_name_here, 8 links, 7 joints
Links:
- added link laser_horiz_velodyne, mass 0.01; visual mesh filename=package://velodyne_description/meshes/VLP16_scan.dae
- added link laser_horiz_velodyne_base_link, mass 0.83; collision cylinder length=0.0717 radius=0.0516; visual mesh filename=package://velodyne_description/meshes/VLP16_base_1.dae
- added link laser_vert_bottom_gaze, mass 1e-5; collision box size=0.1 0.1 0.1; visual mesh filename=package://gazebo_plugins/test/multi_robot_scenario/meshes/l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
- added link laser_vert_top_left_gaze, mass 1e-5; collision box size=0.1 0.1 0.1; visual mesh filename=package://gazebo_plugins/test/multi_robot_scenario/meshes/l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
- added link laser_vert_top_right_gaze, mass 1e-5; collision box size=0.1 0.1 0.1; visual mesh filename=package://gazebo_plugins/test/multi_robot_scenario/meshes/l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
Joints:
- added joint base_laser_vert_bottom_gaze_joint: type fixed, parent base, child laser_vert_bottom_gaze, origin xyz=0.3157894464801903 -0.002068548615034871 0.5099999434059285 rpy=3.1354753 -1.3045001 0.0024658, axis 0 0 1
- added joint base_laser_vert_top_left_gaze_joint: type fixed, parent base, child laser_vert_top_left_gaze, origin xyz=0.3157894464801903 -0.002068548615034871 0.5099999434059285 rpy=3.1354753 -1.3045001 0.0024658, axis 0 0 1
- added joint base_laser_vert_top_right_gaze_joint: type fixed, parent base, child laser_vert_top_right_gaze, origin xyz=0.3157894464801903 -0.002068548615034871 0.5099999434059285 rpy=3.1354753 -1.3045001 0.0024658, axis 0 0 1
- added joint laser_horiz_velodyne_base_mount_joint: type fixed, parent base, child laser_horiz_velodyne_base_link, origin xyz=0.2325416305773505 -0.0001380069427607134 1.920122926231907 rpy=-0.0012068 0.114646 -0.0015308
- added joint laser_horiz_velodyne_base_scan_joint: type fixed, parent laser_horiz_velodyne_base_link, child laser_horiz_velodyne, origin xyz=0 0 0.0377 rpy=0 0 0

File: urdf/robot.xacro (robot description, xacro)
@@ -86,3 +86,13 @@
     <limit effort="1" velocity="1"/>
   </joint>
+<xacro:include filename="$(find gazebo_plugins)/test/multi_robot_scenario/xacro/laser/hokuyo.xacro" />
+<xacro:laser name="laser_vert_bottom_gaze" parent="base" xyz="0.3157894464801903 -0.002068548615034871 0.5099999434059285" rpy="3.1354753 -1.3045001 0.0024658" meshes="package://gazebo_plugins/test/multi_robot_scenario/meshes/laser" />
+<xacro:include filename="$(find gazebo_plugins)/test/multi_robot_scenario/xacro/laser/hokuyo.xacro" />
+<xacro:laser name="laser_vert_top_right_gaze" parent="base" xyz="0.3157894464801903 -0.002068548615034871 0.5099999434059285" rpy="3.1354753 -1.3045001 0.0024658" meshes="package://gazebo_plugins/test/multi_robot_scenario/meshes/laser" />
+<xacro:include filename="$(find gazebo_plugins)/test/multi_robot_scenario/xacro/laser/hokuyo.xacro" />
+<xacro:laser name="laser_vert_top_left_gaze" parent="base" xyz="0.3157894464801903 -0.002068548615034871 0.5099999434059285" rpy="3.1354753 -1.3045001 0.0024658" meshes="package://gazebo_plugins/test/multi_robot_scenario/meshes/laser" />
+<xacro:include filename="$(find velodyne_description)/urdf/VLP-16.urdf.xacro"/>
+<VLP-16 parent="base" name="laser_horiz_velodyne" topic="laser_horiz/packets" hz="10" samples="440" gpu="false">
+<origin xyz="0.2325416305773505 -0.0001380069427607134 1.920122926231907" rpy="-0.0012068 0.114646 -0.0015308" />
+</VLP-16>
 </robot >

Commit message: fixed some location problem

File: urdf/robot.urdf (robot description, URDF)
Before this commit: robot insert_robot_name_here, 13 links, 12 joints
Joints:
- joint base_laser_vert_top_left_gaze_joint: origin xyz=0.3157894464801903 -0.002068548615034871 0.5099999434059285 rpy=3.1354753 -1.3045001 0.0024658 -> xyz=0.2997 0.1531 1.8443 rpy=1.1780 0.6198 1.9560
- joint base_laser_vert_top_right_gaze_joint: origin xyz=0.3157894464801903 -0.002068548615034871 0.5099999434059285 rpy=3.1354753 -1.3045001 0.0024658 -> xyz=0.2978 -0.1450 1.8451 rpy=-1.1760 0.6313 -1.9377
- joint base_to_laser_vert_top_right: origin xyz=0.2978 -0.1450 1.8451 rpy=-1.1760 0.6313 -1.9377 -> (none)

File: urdf/robot.xacro (robot description, xacro)
@@ -20,4 +20,6 @@
     <child link="laser_vert_bottom"/>
   </joint>
+  <xacro:include filename="$(find gazebo_plugins)/test/multi_robot_scenario/xacro/laser/hokuyo.xacro" />
+  <xacro:laser name="laser_vert_bottom_gaze" parent="base" xyz="0.3157894464801903 -0.002068548615034871 0.5099999434059285" rpy="3.1354753 -1.3045001 0.0024658" meshes="package://gazebo_plugins/test/multi_robot_scenario/meshes/laser" />
   <link name="laser_vert_top_right">
     <visual>
@@ -25,4 +27,5 @@
         <box size="0.062 0.062 0.087"/>
       </geometry>
+      <origin xyz="0.2978 -0.1450 1.8451" rpy="-1.1760 0.6313 -1.9377"/>
     </visual>
   </link>
@@ -30,6 +33,7 @@
     <parent link="base"/>
     <child link="laser_vert_top_right"/>
-    <origin xyz="0.2978 -0.1450 1.8451" rpy="-1.1760 0.6313 -1.9377"/>
   </joint>
+  <xacro:include filename="$(find gazebo_plugins)/test/multi_robot_scenario/xacro/laser/hokuyo.xacro" />
+  <xacro:laser name="laser_vert_top_right_gaze" parent="base" xyz="0.2978 -0.1450 1.8451" rpy="-1.1760 0.6313 -1.9377" meshes="package://gazebo_plugins/test/multi_robot_scenario/meshes/laser" />
   <link name="laser_vert_top_left">
     <visual>
@@ -44,4 +48,6 @@
     <child link="laser_vert_top_left"/>
   </joint>
+  <xacro:include filename="$(find gazebo_plugins)/test/multi_robot_scenario/xacro/laser/hokuyo.xacro" />
+  <xacro:laser name="laser_vert_top_left_gaze" parent="base" xyz="0.2997 0.1531 1.8443" rpy="1.1780 0.6198 1.9560" meshes="package://gazebo_plugins/test/multi_robot_scenario/meshes/laser" />
   <link name="laser_horiz">
     <visual>
@@ -56,4 +62,8 @@
     <child link="laser_horiz"/>
   </joint>
+  <xacro:include filename="$(find velodyne_description)/urdf/VLP-16.urdf.xacro"/>
+  <VLP-16 parent="base" name="laser_horiz_velodyne" topic="laser_horiz/packets" hz="10" samples="440" gpu="false">
+        <origin xyz="0.2325416305773505 -0.0001380069427607134 1.920122926231907" rpy="-0.0012068 0.114646 -0.0015308" />
+  </VLP-16>
 <xacro:macro name="xacro_name" params="suffix reflect">
   <link name="wheel_${suffix}">
@@ -86,13 +96,3 @@
     <limit effort="1" velocity="1"/>
   </joint>
-<xacro:include filename="$(find gazebo_plugins)/test/multi_robot_scenario/xacro/laser/hokuyo.xacro" />
-<xacro:laser name="laser_vert_bottom_gaze" parent="base" xyz="0.3157894464801903 -0.002068548615034871 0.5099999434059285" rpy="3.1354753 -1.3045001 0.0024658" meshes="package://gazebo_plugins/test/multi_robot_scenario/meshes/laser" />
-<xacro:include filename="$(find gazebo_plugins)/test/multi_robot_scenario/xacro/laser/hokuyo.xacro" />
-<xacro:laser name="laser_vert_top_right_gaze" parent="base" xyz="0.3157894464801903 -0.002068548615034871 0.5099999434059285" rpy="3.1354753 -1.3045001 0.0024658" meshes="package://gazebo_plugins/test/multi_robot_scenario/meshes/laser" />
-<xacro:include filename="$(find gazebo_plugins)/test/multi_robot_scenario/xacro/laser/hokuyo.xacro" />
-<xacro:laser name="laser_vert_top_left_gaze" parent="base" xyz="0.3157894464801903 -0.002068548615034871 0.5099999434059285" rpy="3.1354753 -1.3045001 0.0024658" meshes="package://gazebo_plugins/test/multi_robot_scenario/meshes/laser" />
-<xacro:include filename="$(find velodyne_description)/urdf/VLP-16.urdf.xacro"/>
-<VLP-16 parent="base" name="laser_horiz_velodyne" topic="laser_horiz/packets" hz="10" samples="440" gpu="false">
-<origin xyz="0.2325416305773505 -0.0001380069427607134 1.920122926231907" rpy="-0.0012068 0.114646 -0.0015308" />
-</VLP-16>
 </robot >
