Commit message: new version of lab4_package for lab5

File: urdf/robot.xacro (robot description, xacro)
@@ -72,5 +72,5 @@
         <cylinder length="0.05" radius="0.2"/>
       </geometry>
-      <origin rpy="${-pi/2} 0.0 0.0" xyz="0.1 ${reflect * -0.4} 0.0"/>
+      <origin rpy="-1.57079632679 0.0 0.0" xyz="-0.1 ${reflect * -0.4} 0.0"/>
     </visual>
   </link>
@@ -88,5 +88,5 @@
         <cylinder length="0.05" radius="0.15"/>
       </geometry>
-      <origin rpy="${-pi/2} 0.0 0.0" xyz="0.1 0.0 0.0"/>
+      <origin rpy="-1.57079632679 0 0" xyz="0.1 0 0"/>
     </visual>
   </link>
