Commit message: finished version of lab5

File: urdf/new.xacro (robot description, xacro)
@@ -7,5 +7,5 @@
 		<parent link="base_link" />
 		<child link="base" />
-		<origin xyz="0.07 0 1.792" rpy="0.0 ${pi} 0.0" />
+		<origin xyz="0.07 0 1.792" rpy="0.0 3.14159265359 0.0" />
 	</joint>
 	<joint name="base_link_imu_joint" type="fixed">

File: urdf/robot.xacro (robot description, xacro)
@@ -78,5 +78,5 @@
     <parent link="base"/>
     <child link="wheel_${suffix}"/>
-    <limit effort="1" velocity="1"/>
+    <limit effort="100" velocity="100"/>
   </joint>
 </xacro:macro>
